File: skytraq_px1125r_kicad.kicad_pcb (KiCad board)
At the start: 2 copper layers, 35.5 x 27.6 mm, 11 parts, among them J1 Conn_01x04, J2 SMA, J3 SH_Conn_01x04, J4 Conn_01x04, U1 Skytraq_PX1125R

Commit message: PX1105
Parts:
- removed U1: Skytraq_PX1125R, RF_GPS:ublox_NEO
- added U2: ~, MySkyTraqFootprints:skytraq_px1105, F.Cu at (124.9, 49.0)
- moved R6 25.9 mm to (123.0, 36.0), turned to 0 degrees
- moved C1 22.9 mm to (132.2, 54.8), turned to -90 degrees
- moved D2 1.09 mm to (117.7, 38.0)
- moved R5 1.09 mm to (123.0, 38.0)
Connections:
- J1 pad 3: GPS_EXTINT -> GPS_BOOT
Routing:
- net GPS_BOOT: track 0.00 -> 49.2 mm, vias 0 -> 1
- net GPS_RXD2: track 10.8 -> 47.8 mm, vias 0 -> 1
- net GPS_EXTINT: track 15.5 -> 0.00 mm, vias 1 -> 0
- net GPS_PPS: track 35.3 -> 50.4 mm
- net GPS_RXD: track 22.6 -> 30.6 mm
- net +3V3: track 68.7 -> 61.4 mm, vias 4 -> 1
- net GPS_TXD: track 20.8 -> 28.0 mm
- net GPS_RST: track 11.2 -> 12.6 mm, vias 0 -> 2
- net Net-(J2-In): track 12.9 -> 11.5 mm
- net GND: vias 0 -> 15
Other:
- board text added: "BOOT"
- board text added: "SkyTraq PX1105R"
- board text removed: "ODO"
- board text removed: "SkyTraq PX1125R"
