File: skytraq_px1125r_kicad.kicad_sch (KiCad schematic)
At the start: 47 parts, among them J1 JST_GH_1.25_6P, J2 SMA, J3 JST_GH_1.25_6P, J5 Conn_01x06, J7 Conn_01x06, U1 Skytraq_PX1125R, U2 RV-3032, U3 LIS3MDL, U5 SkyTraq_PX1105, U6 AMS1117-3.3

Commit message: 36x36 for flight controllers
Parts:
- removed C6: 22uF, Capacitor_Tantalum_SMD:CP_EIA-3216-18_Kemet-A, symbol Device:C_Polarized
- removed H1: MountingHole, MountingHole:MountingHole_3.2mm_M3, symbol Mechanical:MountingHole
- removed J5, J7: Conn_01x06, Connector_PinHeader_2.54mm:PinHeader_1x06_P2.54mm_Vertical, symbol Connector_Generic:Conn_01x06
- removed R8, R9: 0, Resistor_SMD:R_0603_1608Metric, symbol Device:R
- added C11, C13, C14, C16, C6: 10uF, Capacitor_SMD:C_0603_1608Metric, symbol Device:C
- added C12, C15: 100nF, Capacitor_SMD:C_0402_1005Metric, symbol Device:C
- added D4, D5: D_Schottky, Diode_SMD:D_SOD-323, symbol Device:D_Schottky
- added FB2: FerriteBead, Inductor_SMD:L_0805_2012Metric, symbol Device:FerriteBead
- added H1: MountingHole_Pad, MyFootprints:MountingHole_3.2mm_M3_Pad, symbol Mechanical:MountingHole_Pad
- added J5: USB_C_Receptacle_USB2.0_16P, footprint:USB-C_SMD-TYPE-C-31-M-12_1, symbol Connector:USB_C_Receptacle_USB2.0_16P
- added R15: 1k, Resistor_SMD:R_0402_1005Metric, symbol Device:R
- added R16: 22k, Resistor_SMD:R_0402_1005Metric, symbol Device:R
- added R17: 47k, Resistor_SMD:R_0402_1005Metric, symbol Device:R
- added R20, R21: 5.1k, Resistor_SMD:R_0402_1005Metric, symbol Device:R
- added U4: CP2102N-A02-GQFN20R, footprint:QFN-20_L3.0-W3.0-P0.50-BL-EP1.7_EFM8BB21F16G, symbol CP2102N-A02-GQFN20R:CP2102N-A02-GQFN20R
- added U7: USBLC6-2SC6, Package_TO_SOT_SMD:SOT-23-6, symbol Power_Protection:USBLC6-2SC6
- BT1: now not fitted
- C1, C3: LCSC C19702 -> C2959727; Note Low ESR! X7R -> (none)
- C10: LCSC C1525 -> C71629; Note Low ESR! X7R -> (none)
- C2: footprint Capacitor_SMD:C_0603_1608Metric -> Capacitor_SMD:C_0805_2012Metric_Pad1.18x1.45mm_HandSolder; LCSC C1671 -> (none)
- C23: LCSC C19702 -> C2959727; now not fitted; now left out of the parts list
- C4: value 100nF -> 10uF; footprint Capacitor_SMD:C_0805_2012Metric_Pad1.18x1.45mm_HandSolder -> Capacitor_SMD:C_0603_1608Metric; LCSC (none) -> C2959727; now in the parts list
- C5: footprint Capacitor_SMD:C_0805_2012Metric_Pad1.18x1.45mm_HandSolder -> Capacitor_SMD:C_0603_1608Metric; LCSC (none) -> C2959727; now in the parts list
- C7: LCSC C19702 -> C2959727
- C8, C9: LCSC C1525 -> C71629; now not fitted; now left out of the parts list
- D1: Note PWR -> (none)
- D2: Note PPS -> (none)
- D6: LCSC C22452 -> C7380001
- H2, H3, H4: value MountingHole -> MountingHole_Pad; footprint MountingHole:MountingHole_3.2mm_M3 -> MyFootprints:MountingHole_3.2mm_M3_Pad; symbol Mechanical:MountingHole -> Mechanical:MountingHole_Pad
- J1, J3: LCSC (none) -> C3029381
- J2: footprint footprint:SMA-SMD_BWSMA-KE-P001_Symmetric -> footprint:SMA-SMD_BWSMA-KE-P001; now left out of the parts list
- R1, R10, R14, R2, R3, R6: footprint Resistor_SMD:R_0603_1608Metric -> Resistor_SMD:R_0402_1005Metric; LCSC C25804 -> C25744
- R11: footprint Resistor_SMD:R_0603_1608Metric -> Resistor_SMD:R_0402_1005Metric; LCSC C25804 -> C25744; now not fitted; now left out of the parts list
- R12, R13, R4, R5: footprint Resistor_SMD:R_0603_1608Metric -> Resistor_SMD:R_0402_1005Metric; LCSC C21190 -> C11702
- R7: footprint Resistor_SMD:R_0603_1608Metric -> Resistor_SMD:R_0805_2012Metric_Pad1.20x1.40mm_HandSolder; LCSC C22859 -> (none)
- U1: symbol MySymbols:Skytraq_PX1125R -> MySymbolsGlobal:Skytraq_PX1125R
- U2: symbol MySymbols:RV-3032 -> MySymbolsGlobal:RV-3032
- U3: LCSC (none) -> C478483; now not fitted; now left out of the parts list
- U5: symbol MySkyTraqSymbols:SkyTraq_PX1105 -> MySymbolsGlobal:SkyTraq_PX1105
- U6: LCSC (none) -> C880752
Connections:
- net +3V3: now also C3.1, C4.2, C5.2, JP1.1 (A), U1.22 (V_BCKP), U5.6 (V_BCKP), C13.2, C16.1, C6.2; no longer C5.1, JP1.3 (B)
- net +5V: now also D4.1 (K), D5.1 (K); no longer J1.1 (Pin_1), J3.1 (Pin_1)
- net GND: now also C4.1, C5.1, H2.1, H3.1, H4.1, JP1.3 (B), C11.1, C12.2, C13.1, C14.1, C15.2, C16.2, C6.1, H1.1, J5.A1 (GND), J5.A12 (GND), J5.B1 (GND), J5.B12 (GND), J5.S1 (SHIELD), R17.2, R20.2, R21.2, U4.12 (GND), U4.21 (EP), U4.3 (GND), U7.2 (GND); no longer C4.2, C5.2
- net GPS_RX: now also U4.18 (TXD)
- net GPS_TX: now also U4.17 (RXD)
- net VBAT: no longer JP1.1 (A)
- net at U3.9 (SDO/SA1): now also JP1.2 (C)
- removed net GPS_V_BCKP: C3.1, C4.1, JP1.2 (C), U1.22 (V_BCKP), U5.6 (V_BCKP)
- new net: R16.2, R17.1, U4.8 (VBUS)
- new net: FB2.1, J5.A4 (VBUS), J5.A9 (VBUS), J5.B4 (VBUS), J5.B9 (VBUS), U7.5 (VBUS)
- new net: J5.A5 (CC1), R20.1
- new net: R15.2, U4.9 (~{RST})
- new net: J5.A6 (D+), J5.B6 (D+), U7.3 (I/O2)
- new net: J5.A7 (D-), J5.B7 (D-), U7.1 (I/O1)
- new net: J5.B5 (CC2), R21.1
- new net +3V3_USB: C14.2, C15.1, R15.1, U4.6 (VDD)
- new net +5V_IN: D5.2 (A), J1.1 (Pin_1), J3.1 (Pin_1)
- new net +5V_USB: C11.2, C12.1, D4.2 (A), FB2.2, R16.1, U4.7 (VREGIN)
- new net USB_DN: U4.5 (D-), U7.6 (I/O1)
- new net USB_DP: U4.4 (D+), U7.4 (I/O2)
- no-connect marks 16 -> 27
Other:
- moved on the sheet: C1, C10, C2, C3, C7, D1, D2, D3, D6, J1, J2, J3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
